Commit message: fix(examples): add inertial tags and visual geometry to robot_arm.urdf
Required for MuJoCo compatibility. Added mass/inertia to all links
and simple box visual meshes so the arm renders in the sim viewport.

File: examples/robot_arm.urdf (robot description, URDF)
Before this commit: robot dummy_arm, 8 links, 7 joints
Links:
- link base_link: mass None -> 1.0; geometry visual box size=0.2 0.2 0.1
- link l1: mass None -> 0.8; geometry visual box size=0.08 0.08 0.3
- link l2: mass None -> 0.7; geometry visual box size=0.07 0.07 0.3
- link l3: mass None -> 0.6; geometry visual box size=0.06 0.06 0.24
- link l4: mass None -> 0.5; geometry visual box size=0.05 0.05 0.2
- link l5: mass None -> 0.4; geometry visual box size=0.04 0.04 0.16
- link l6: mass None -> 0.3; geometry visual box size=0.03 0.03 0.12
- link l7: mass None -> 0.2; geometry visual box size=0.03 0.03 0.08
Joints:
- joint j1: limit (none) -> lower=-3.14 upper=3.14 effort=10 velocity=1; origin (none) -> xyz=0 0 0.15 rpy=0 0 0
- joint j2: limit (none) -> lower=-2.0 upper=2.0 effort=10 velocity=1; origin (none) -> xyz=0 0 0.3 rpy=0 0 0
- joint j3: limit (none) -> lower=-2.0 upper=2.0 effort=10 velocity=1; origin (none) -> xyz=0 0 0.3 rpy=0 0 0
- joint j4: limit (none) -> lower=-1.5 upper=1.5 effort=10 velocity=1; origin (none) -> xyz=0 0 0.24 rpy=0 0 0
- joint j5: limit (none) -> lower=-1.5 upper=1.5 effort=10 velocity=1; origin (none) -> xyz=0 0 0.2 rpy=0 0 0
- joint j6: limit (none) -> lower=-1.5 upper=1.5 effort=10 velocity=1; origin (none) -> xyz=0 0 0.16 rpy=0 0 0
- joint j7: limit (none) -> lower=-1.5 upper=1.5 effort=10 velocity=1; origin (none) -> xyz=0 0 0.12 rpy=0 0 0
